File: KiCad_PCB_Files/Kicad Project/Arduino_Spot_Welder.sch (KiCad schematic (older format))
At the start: 55 parts, among them P1 MCP1407, P2 GND_con, P3 GND_con, P4 GND_con, P5 GND_con, P6 OLED_Display, Q1 IRFB_7430, Q2 IRFB_7430, Q3 IRFB_7430, Q4 IRFB_7430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

Commit message: Add files via upload
Parts:
- ENC1: value ALPS-STEC12E08 -> Bourns_PEC11L
- P3, P5: value GND_con -> AutoPulse
Changed lines of the file:
@@
 P 4350 3450
 F 0 "P3" H 4350 3600 50  0000 C CNN
-F 1 "GND_con" V 4450 3450 50  0000 C CNN
+F 1 "AutoPulse" V 4450 3450 50  0000 C CNN
 F 2 "Pin_Headers:Pin_Header_Straight_1x02_Pitch2.54mm" H 4350 3450 50  0001 C CNN
 F 3 "" H 4350 3450 50  0000 C CNN
@@
 P 8325 1350
 F 0 "P5" H 8325 1500 50  0000 C CNN
-F 1 "GND_con" V 8425 1350 50  0000 C CNN
+F 1 "AutoPulse" V 8425 1350 50  0000 C CNN
 F 2 "Pin_Headers:Pin_Header_Straight_1x02_Pitch2.54mm" H 8325 1350 50  0001 C CNN
 F 3 "" H 8325 1350 50  0000 C CNN
@@
 P 3875 1625
 F 0 "ENC1" H 3875 2000 60  0000 C CNN
-F 1 "ALPS-STEC12E08" H 3875 2125 60  0000 C CNN
+F 1 "Bourns_PEC11L" H 3875 2125 60  0000 C CNN
 F 2 "Rotary-Encoders:ALPS_STEC12E08" H 3875 1625 60  0001 C CNN
 F 3 "" H 3875 1625 60  0000 C CNN
