File: KiCad_PCB_Files/Kicad Project/Kicad Project V3.3/Arduino_Spot_Welder.sch (KiCad schematic (older format))
At the start: 58 parts, among them P1 MCP1407, P2 GND_con, P3 AutoPulse, P4 GND_con, P5 AutoPulse, P6 OLED_Display, P7 V IN, Q1 IRFB_7430, Q2 IRFB_7430, Q3 IRFB_7430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

Commit message: using stm32f030 mcu
Parts:
- C1, C3, C4, C6: symbol C -> Arduino_Spot_Welder-rescue:C
- C2, C5: symbol CP -> Arduino_Spot_Welder-rescue:CP
- D1, TVS1, TVS2, TVS3, TVS4, TVS5: symbol D -> Arduino_Spot_Welder-rescue:D
- D3: symbol ZENER -> Arduino_Spot_Welder-rescue:ZENER
- D4: symbol D_Schottky_x2_Serial_AKC -> Arduino_Spot_Welder-rescue:D_Schottky_x2_Serial_AKC
- ENC1: symbol ALPS-STEC12E08 -> Arduino_Spot_Welder-rescue:ALPS-STEC12E08
- Foot_Switch1, P2, P3, P4, P5, P7: symbol CONN_01X02 -> Arduino_Spot_Welder-rescue:CONN_01X02
- Mosfet_CTRL1, Mosfet_CTRL2: symbol CONN_01X08 -> Arduino_Spot_Welder-rescue:CONN_01X08
- P1: symbol DIL8 -> Arduino_Spot_Welder-rescue:DIL8
- P6: symbol CONN_01X04 -> Arduino_Spot_Welder-rescue:CONN_01X04
- Q1, Q2, Q3, Q4, Q5, Q6, Q7, Q8: symbol IRF540N -> Arduino_Spot_Welder-rescue:IRF540N
- R1, R10, R11, R12, R13, R14, R15, R16, R17, R18, R19, R2, R20, R21, R22, R23, R24, R3, R4, R5, R6, R7, R8, R9: symbol R -> Arduino_Spot_Welder-rescue:R
- U1: symbol arduino_mini -> Arduino_Spot_Welder-rescue:arduino_mini
